File: nixie_tube_board/nixie_tube_board.kicad_pcb (KiCad board)
At the start: 2 copper layers, 127 x 45.7 mm, 46 parts, among them J1 Conn_02x05_Odd_Even, J2 Conn_02x05_Odd_Even, Q1 MPSA42, Q2 MPSA42, Q3 MPSA42, Q4 MPSA42, Q5 MPSA92, Q6 MPSA92, Q7 MPSA92, Q8 MPSA92, Q9 MPSA42, U1 74HC595, U2 74HC595, U3 74141, U4 74141, U5 74141, U6 74141

Commit message: Fix mpsa92 orientation
Parts:
- moved Q5 2.54 mm to (154.9, 116.8), turned to 0 degrees
- moved Q6 2.54 mm to (132.1, 116.8), turned to 0 degrees
- moved Q7 2.54 mm to (99.1, 116.8), turned to 0 degrees
- moved Q8 2.54 mm to (76.2, 116.8), turned to 0 degrees
Connections:
- Q5 pad 1: Net-(Q5-Pad1) -> +170V
- Q5 pad 3: +170V -> Net-(R9-Pad1)
- Q6 pad 1: Net-(Q6-Pad1) -> +170V
- Q6 pad 3: +170V -> Net-(Q6-Pad3)
- Q7 pad 1: Net-(Q7-Pad1) -> +170V
- Q7 pad 3: +170V -> Net-(Q7-Pad3)
- Q8 pad 1: Net-(Q8-Pad1) -> +170V
- Q8 pad 3: +170V -> Net-(Q8-Pad3)
- R10 pad 1: Net-(Q6-Pad1) -> Net-(Q6-Pad3)
- R11 pad 1: Net-(Q7-Pad1) -> Net-(Q7-Pad3)
- R12 pad 1: Net-(Q8-Pad1) -> Net-(Q8-Pad3)
- R9 pad 1: Net-(Q5-Pad1) -> Net-(R9-Pad1)
Routing:
- net Net-(Q8-Pad3): track 0.00 -> 4.38 mm
- net Net-(Q8-Pad1): track 4.38 -> 0.00 mm
- net Net-(Q7-Pad3): track 0.00 -> 4.38 mm
- net Net-(Q7-Pad1): track 4.38 -> 0.00 mm
- net Net-(R9-Pad1): track 0.00 -> 4.34 mm
- net Net-(Q5-Pad1): track 4.34 -> 0.00 mm
- net Net-(Q6-Pad3): track 0.00 -> 4.34 mm
- net Net-(Q6-Pad1): track 4.34 -> 0.00 mm
Changed lines of the file:
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@@
   (title_block
     (title "Nixie Clock Tube Board")
-    (date "2022-01-29")
-    (rev "1")
+    (date "2022-02-10")
+    (rev "2")
   )
   (layers
@@
   (net 65 "Net-(Q4-Pad1)")
   (net 66 "Net-(Q4-Pad3)")
-  (net 67 "Net-(Q5-Pad1)")
-  (net 68 "Net-(Q6-Pad1)")
-  (net 69 "Net-(Q7-Pad1)")
-  (net 70 "Net-(Q8-Pad1)")
+  (net 67 "Net-(R9-Pad1)")
+  (net 68 "Net-(Q6-Pad3)")
+  (net 69 "Net-(Q7-Pad3)")
+  (net 70 "Net-(Q8-Pad3)")
   (net 71 "Net-(U1-Pad15)")
   (net 72 "Net-(U1-Pad7)")
@@
   )
   (footprint "Package_TO_SOT_THT:TO-92_Inline" (layer "F.Cu")
-    (at 157.48 116.84 180)
+    (at 154.94 116.84)
     (descr "TO-92 leads in-line, narrow, oval pads, drill 0.75mm (see NXP sot054_po.pdf)")
     (tags "to-92 sc-43 sc-43a sot54 PA33 transistor")
@@
     (fp_arc (start -0.483625 1.753625) (mid -1.021221 -0.949055) (end 1.27 -2.48) (layer "F.Fab") (width 0.1))
     (fp_arc (start 1.27 -2.48) (mid 3.561221 -0.949055) (end 3.023625 1.753625) (layer "F.Fab") (width 0.1))
-    (pad "1" thru_hole rect locked (at 0 0 180) (size 1.05 1.5) (drill 0.75) (layers *.Cu *.Mask)
-      (net 67 "Net-(Q5-Pad1)") (pinfunction "E") (pintype "passive"))
-    (pad "2" thru_hole oval locked (at 1.27 0 180) (size 1.05 1.5) (drill 0.75) (layers *.Cu *.Mask)
+    (pad "1" thru_hole rect locked (at 0 0) (size 1.05 1.5) (drill 0.75) (layers *.Cu *.Mask)
+      (net 74 "+170V") (pinfunction "E") (pintype "passive"))
+    (pad "2" thru_hole oval locked (at 1.27 0) (size 1.05 1.5) (drill 0.75) (layers *.Cu *.Mask)
       (net 61 "Net-(Q1-Pad3)") (pinfunction "B") (pintype "input"))
-    (pad "3" thru_hole oval locked (at 2.54 0 180) (size 1.05 1.5) (drill 0.75) (layers *.Cu *.Mask)
-      (net 74 "+170V") (pinfunction "C") (pintype "passive"))
+    (pad "3" thru_hole oval locked (at 2.54 0) (size 1.05 1.5) (drill 0.75) (layers *.Cu *.Mask)
+      (net 67 "Net-(R9-Pad1)") (pinfunction "C") (pintype "passive"))
     (model "${KICAD6_3DMODEL_DIR}/Package_TO_SOT_THT.3dshapes/TO-92_Inline.wrl"
       (offset (xyz 0 0 0))
@@
     (fp_line (start 6.96 -1.25) (end 0.66 -1.25) (layer "F.Fab") (width 0.1))
     (pad "1" thru_hole circle locked (at 0 0 90) (size 1.6 1.6) (drill 0.8) (layers *.Cu *.Mask)
-      (net 68 "Net-(Q6-Pad1)") (pintype "passive"))
+      (net 68 "Net-(Q6-Pad3)") (pintype "passive"))
     (pad "2" thru_hole oval locked (at 7.62 0 90) (size 1.6 1.6) (drill 0.8) (layers *.Cu *.Mask)
       (net 30 "Net-(N2-PadA)") (pintype "passive"))
@@
     (fp_line (start 7.62 0) (end 6.96 0) (layer "F.Fab") (width 0.1))
     (pad "1" thru_hole circle locked (at 0 0 90) (size 1.6 1.6) (drill 0.8) (layers *.Cu *.Mask)
-      (net 67 "Net-(Q5-Pad1)") (pintype "passive"))
+      (net 67 "Net-(R9-Pad1)") (pintype "passive"))
     (pad "2" thru_hole oval locked (at 7.62 0 90) (size 1.6 1.6) (drill 0.8) (layers *.Cu *.Mask)
       (net 5 "Net-(N1-PadA)") (pintype "passive"))
@@
   )
   (footprint "Package_TO_SOT_THT:TO-92_Inline" (layer "F.Cu")
-    (at 78.74 116.84 180)
+    (at 76.2 116.84)
     (descr "TO-92 leads in-line, narrow, oval pads, drill 0.75mm (see NXP sot054_po.pdf)")
     (tags "to-92 sc-43 sc-43a sot54 PA33 transistor")
@@
     (fp_arc (start -0.483625 1.753625) (mid -1.021221 -0.949055) (end 1.27 -2.48) (layer "F.Fab") (width 0.1))
     (fp_arc (start 1.27 -2.48) (mid 3.561221 -0.949055) (end 3.023625 1.753625) (layer "F.Fab") (width 0.1))
-    (pad "1" thru_hole rect locked (at 0 0 180) (size 1.05 1.5) (drill 0.75) (layers *.Cu *.Mask)
-      (net 70 "Net-(Q8-Pad1)") (pinfunction "E") (pintype "passive"))
-    (pad "2" thru_hole oval locked (at 1.27 0 180) (size 1.05 1.5) (drill 0.75) (layers *.Cu *.Mask)
+    (pad "1" thru_hole rect locked (at 0 0) (size 1.05 1.5) (drill 0.75) (layers *.Cu *.Mask)
+      (net 74 "+170V") (pinfunction "E") (pintype "passive"))
+    (pad "2" thru_hole oval locked (at 1.27 0) (size 1.05 1.5) (drill 0.75) (layers *.Cu *.Mask)
       (net 66 "Net-(Q4-Pad3)") (pinfunction "B") (pintype "input"))
-    (pad "3" thru_hole oval locked (at 2.54 0 180) (size 1.05 1.5) (drill 0.75) (layers *.Cu *.Mask)
-      (net 74 "+170V") (pinfunction "C") (pintype "passive"))
+    (pad "3" thru_hole oval locked (at 2.54 0) (size 1.05 1.5) (drill 0.75) (layers *.Cu *.Mask)
+      (net 70 "Net-(Q8-Pad3)") (pinfunction "C") (pintype "passive"))
     (model "${KICAD6_3DMODEL_DIR}/Package_TO_SOT_THT.3dshapes/TO-92_Inline.wrl"
       (offset (xyz 0 0 0))
@@
     (fp_line (start 0.66 -1.25) (end 0.66 1.25) (layer "F.Fab") (width 0.1))
     (pad "1" thru_hole circle locked (at 0 0 90) (size 1.6 1.6) (drill 0.8) (layers *.Cu *.Mask)
-      (net 69 "Net-(Q7-Pad1)") (pintype "passive"))
+      (net 69 "Net-(Q7-Pad3)") (pintype "passive"))
     (pad "2" thru_hole oval locked (at 7.62 0 90) (size 1.6 1.6) (drill 0.8) (layers *.Cu *.Mask)
       (net 40 "Net-(N3-PadA)") (pintype "passive"))
@@
   )
   (footprint "Package_TO_SOT_THT:TO-92_Inline" (layer "F.Cu")
-    (at 134.62 116.84 180)
+    (at 132.08 116.84)
     (descr "TO-92 leads in-line, narrow, oval pads, drill 0.75mm (see NXP sot054_po.pdf)")
     (tags "to-92 sc-43 sc-43a sot54 PA33 transistor")
@@
     (fp_arc (start -0.483625 1.753625) (mid -1.021221 -0.949055) (end 1.27 -2.48) (layer "F.Fab") (width 0.1))
     (fp_arc (start 1.27 -2.48) (mid 3.561221 -0.949055) (end 3.023625 1.753625) (layer "F.Fab") (width 0.1))
-    (pad "1" thru_hole rect locked (at 0 0 180) (size 1.05 1.5) (drill 0.75) (layers *.Cu *.Mask)
-      (net 68 "Net-(Q6-Pad1)") (pinfunction "E") (pintype "passive"))
-    (pad "2" thru_hole oval locked (at 1.27 0 180) (size 1.05 1.5) (drill 0.75) (layers *.Cu *.Mask)
+    (pad "1" thru_hole rect locked (at 0 0) (size 1.05 1.5) (drill 0.75) (layers *.Cu *.Mask)
+      (net 74 "+170V") (pinfunction "E") (pintype "passive"))
+    (pad "2" thru_hole oval locked (at 1.27 0) (size 1.05 1.5) (drill 0.75) (layers *.Cu *.Mask)
       (net 62 "Net-(Q2-Pad3)") (pinfunction "B") (pintype "input"))
-    (pad "3" thru_hole oval locked (at 2.54 0 180) (size 1.05 1.5) (drill 0.75) (layers *.Cu *.Mask)
-      (net 74 "+170V") (pinfunction "C") (pintype "passive"))
+    (pad "3" thru_hole oval locked (at 2.54 0) (size 1.05 1.5) (drill 0.75) (layers *.Cu *.Mask)
+      (net 68 "Net-(Q6-Pad3)") (pinfunction "C") (pintype "passive"))
     (model "${KICAD6_3DMODEL_DIR}/Package_TO_SOT_THT.3dshapes/TO-92_Inline.wrl"
       (offset (xyz 0 0 0))
@@
   )
   (footprint "Package_TO_SOT_THT:TO-92_Inline" (layer "F.Cu")
-    (at 101.6 116.84 180)
+    (at 99.06 116.84)
     (descr "TO-92 leads in-line, narrow, oval pads, drill 0.75mm (see NXP sot054_po.pdf)")
     (tags "to-92 sc-43 sc-43a sot54 PA33 transistor")
@@
     (fp_arc (start 1.27 -2.48) (mid 3.561221 -0.949055) (end 3.023625 1.753625) (layer "F.Fab") (width 0.1))
     (fp_arc (start -0.483625 1.753625) (mid -1.021221 -0.949055) (end 1.27 -2.48) (layer "F.Fab") (width 0.1))
-    (pad "1" thru_hole rect locked (at 0 0 180) (size 1.05 1.5) (drill 0.75) (layers *.Cu *.Mask)
-      (net 69 "Net-(Q7-Pad1)") (pinfunction "E") (pintype "passive"))
-    (pad "2" thru_hole oval locked (at 1.27 0 180) (size 1.05 1.5) (drill 0.75) (layers *.Cu *.Mask)
+    (pad "1" thru_hole rect locked (at 0 0) (size 1.05 1.5) (drill 0.75) (layers *.Cu *.Mask)
+      (net 74 "+170V") (pinfunction "E") (pintype "passive"))
+    (pad "2" thru_hole oval locked (at 1.27 0) (size 1.05 1.5) (drill 0.75) (layers *.Cu *.Mask)
       (net 64 "Net-(Q3-Pad3)") (pinfunction "B") (pintype "input"))
-    (pad "3" thru_hole oval locked (at 2.54 0 180) (size 1.05 1.5) (drill 0.75) (layers *.Cu *.Mask)
-      (net 74 "+170V") (pinfunction "C") (pintype "passive"))
+    (pad "3" thru_hole oval locked (at 2.54 0) (size 1.05 1.5) (drill 0.75) (layers *.Cu *.Mask)
+      (net 69 "Net-(Q7-Pad3)") (pinfunction "C") (pintype "passive"))
     (model "${KICAD6_3DMODEL_DIR}/Package_TO_SOT_THT.3dshapes/TO-92_Inline.wrl"
       (offset (xyz 0 0 0))
@@
     (fp_line (start 6.96 -1.25) (end 0.66 -1.25) (layer "F.Fab") (width 0.1))
     (pad "1" thru_hole circle locked (at 0 0 90) (size 1.6 1.6) (drill 0.8) (layers *.Cu *.Mask)
-      (net 70 "Net-(Q8-Pad1)") (pintype "passive"))
+      (net 70 "Net-(Q8-Pad3)") (pintype "passive"))
     (pad "2" thru_hole oval locked (at 7.62 0 90) (size 1.6 1.6) (drill 0.8) (layers *.Cu *.Mask)
       (net 51 "Net-(N4-PadA)") (pintype "passive"))
