File: nixie_tube_board/nixie_tube_board.kicad_sch (KiCad schematic)
At the start: 46 parts, among them J1 Conn_02x05_Odd_Even, J2 Conn_02x05_Odd_Even, Q1 MPSA42, Q2 MPSA42, Q3 MPSA42, Q4 MPSA42, Q5 MPSA92, Q6 MPSA92, Q7 MPSA92, Q8 MPSA92, Q9 MPSA42, U1 74HC595, U2 74HC595, U3 74141, U4 74141, U5 74141, U6 74141

Commit message: Add title/date/revision
Other:
- title: (none) -> Nixie Clock Tube Board
Changed lines of the file:
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@@
 (kicad_sch (version 20211123) (generator eeschema)
   (paper "A4")
+  (title_block
+    (title "Nixie Clock Tube Board")
+    (date "2022-01-29")
+    (rev "1")
+  )
   (junction (at 156.21 147.32) (diameter 0) (color 0 0 0 0)
   )

Commit message: Fix mpsa92 orientation
Connections:
- net +170V: now also Q5.1 (E), Q6.1 (E), Q7.1 (E), Q8.1 (E); no longer Q5.3 (C), Q6.3 (C), Q7.3 (C), Q8.3 (C)
- net at R9.1: now also Q5.3 (C); no longer Q5.1 (E)
- net at R10.1: now also Q6.3 (C); no longer Q6.1 (E)
- net at R11.1: now also Q7.3 (C); no longer Q7.1 (E)
- net at R12.1: now also Q8.3 (C); no longer Q8.1 (E)
Changed lines of the file:
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@@
   (title_block
     (title "Nixie Clock Tube Board")
-    (date "2022-01-29")
-    (rev "1")
+    (date "2022-02-10")
+    (rev "2")
   )
   (junction (at 156.21 147.32) (diameter 0) (color 0 0 0 0)
@@
     (pin "3")
   )
-  (symbol (lib_id "Transistor_BJT:MPSA92") (at 153.67 33.02 0) (unit 1)
-    (in_bom yes) (on_board yes)
-    (property "Reference" "Q5" (id 0) (at 158.5214 31.8516 0)
-      (effects (font (size 1.27 1.27)) (justify left))
-    )
-    (property "Value" "MPSA92" (id 1) (at 158.5214 34.163 0)
-      (effects (font (size 1.27 1.27)) (justify left))
-    )
-    (property "Footprint" "Package_TO_SOT_THT:TO-92_Inline" (id 2) (at 158.75 34.925 0)
+  (symbol (lib_id "Transistor_BJT:MPSA92") (at 153.67 33.02 0) (mirror x) (unit 1)
+    (in_bom yes) (on_board yes)
+    (property "Reference" "Q5" (id 0) (at 158.5214 34.1884 0)
+      (effects (font (size 1.27 1.27)) (justify left))
+    )
+    (property "Value" "MPSA92" (id 1) (at 158.5214 31.877 0)
+      (effects (font (size 1.27 1.27)) (justify left))
+    )
+    (property "Footprint" "Package_TO_SOT_THT:TO-92_Inline" (id 2) (at 158.75 31.115 0)
       (effects (font (size 1.27 1.27) italic) (justify left) hide)
     )
@@
     (pin "1")
   )
-  (symbol (lib_id "Transistor_BJT:MPSA92") (at 153.67 74.93 0) (unit 1)
-    (in_bom yes) (on_board yes)
-    (property "Reference" "Q6" (id 0) (at 158.5214 73.7616 0)
-      (effects (font (size 1.27 1.27)) (justify left))
-    )
-    (property "Value" "MPSA92" (id 1) (at 158.5214 76.073 0)
-      (effects (font (size 1.27 1.27)) (justify left))
-    )
-    (property "Footprint" "Package_TO_SOT_THT:TO-92_Inline" (id 2) (at 158.75 76.835 0)
+  (symbol (lib_id "Transistor_BJT:MPSA92") (at 153.67 74.93 0) (mirror x) (unit 1)
+    (in_bom yes) (on_board yes)
+    (property "Reference" "Q6" (id 0) (at 158.5214 76.0984 0)
+      (effects (font (size 1.27 1.27)) (justify left))
+    )
+    (property "Value" "MPSA92" (id 1) (at 158.5214 73.787 0)
+      (effects (font (size 1.27 1.27)) (justify left))
+    )
+    (property "Footprint" "Package_TO_SOT_THT:TO-92_Inline" (id 2) (at 158.75 73.025 0)
       (effects (font (size 1.27 1.27) italic) (justify left) hide)
     )
@@
     (pin "1")
   )
-  (symbol (lib_id "Transistor_BJT:MPSA92") (at 153.67 116.84 0) (unit 1)
-    (in_bom yes) (on_board yes)
-    (property "Reference" "Q7" (id 0) (at 158.5214 115.6716 0)
-      (effects (font (size 1.27 1.27)) (justify left))
-    )
-    (property "Value" "MPSA92" (id 1) (at 158.5214 117.983 0)
-      (effects (font (size 1.27 1.27)) (justify left))
-    )
-    (property "Footprint" "Package_TO_SOT_THT:TO-92_Inline" (id 2) (at 158.75 118.745 0)
+  (symbol (lib_id "Transistor_BJT:MPSA92") (at 153.67 116.84 0) (mirror x) (unit 1)
+    (in_bom yes) (on_board yes)
+    (property "Reference" "Q7" (id 0) (at 158.5214 118.0084 0)
+      (effects (font (size 1.27 1.27)) (justify left))
+    )
+    (property "Value" "MPSA92" (id 1) (at 158.5214 115.697 0)
+      (effects (font (size 1.27 1.27)) (justify left))
+    )
+    (property "Footprint" "Package_TO_SOT_THT:TO-92_Inline" (id 2) (at 158.75 114.935 0)
       (effects (font (size 1.27 1.27) italic) (justify left) hide)
     )
@@
     (pin "1")
   )
-  (symbol (lib_id "Transistor_BJT:MPSA92") (at 153.67 158.75 0) (unit 1)
-    (in_bom yes) (on_board yes)
-    (property "Reference" "Q8" (id 0) (at 158.5214 157.5816 0)
-      (effects (font (size 1.27 1.27)) (justify left))
-    )
-    (property "Value" "MPSA92" (id 1) (at 158.5214 159.893 0)
-      (effects (font (size 1.27 1.27)) (justify left))
-    )
-    (property "Footprint" "Package_TO_SOT_THT:TO-92_Inline" (id 2) (at 158.75 160.655 0)
+  (symbol (lib_id "Transistor_BJT:MPSA92") (at 153.67 158.75 0) (mirror x) (unit 1)
+    (in_bom yes) (on_board yes)
+    (property "Reference" "Q8" (id 0) (at 158.5214 159.9184 0)
+      (effects (font (size 1.27 1.27)) (justify left))
+    )
+    (property "Value" "MPSA92" (id 1) (at 158.5214 157.607 0)
+      (effects (font (size 1.27 1.27)) (justify left))
+    )
+    (property "Footprint" "Package_TO_SOT_THT:TO-92_Inline" (id 2) (at 158.75 156.845 0)
       (effects (font (size 1.27 1.27) italic) (justify left) hide)
     )
