File: nixie_main_board/nixie_main_board.kicad_pcb (KiCad board)
At the start: 2 copper layers, 127 x 45.7 mm, 48 parts, among them J1 Conn_02x05_Odd_Even, J2 Conn_02x05_Odd_Even, J3 USB_C_Receptacle_USB2.0, J4 Conn_01x02_Male, J5 AVR-ISP-6, J6 Conn_01x01_Male, Q1 BC557, Q2 IRL640, SW1 RotaryEncoder_Switch, SW2 SW_Push, SW3 SW_Push, U1 ATmega328P-PU, U2 MC34063AP, U5 DS3231M, Y1 16 MHz

Commit message: Fix sense resistor values
Parts:
- R1, R11, R12, R13, R14: value 0.2 -> 1
Changed lines of the file:
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@@
       (effects (font (size 1 1) (thickness 0.15)))
     )
-    (fp_text value "0.2" (at 3.81 2.37) (layer "F.Fab")
+    (fp_text value "1" (at 3.81 2.37) (layer "F.Fab")
       (effects (font (size 1 1) (thickness 0.15)))
     )
@@
       (effects (font (size 1 1) (thickness 0.15)))
     )
-    (fp_text value "0.2" (at 3.81 2.37) (layer "F.Fab")
+    (fp_text value "1" (at 3.81 2.37) (layer "F.Fab")
       (effects (font (size 1 1) (thickness 0.15)))
     )
@@
       (effects (font (size 1 1) (thickness 0.15)))
     )
-    (fp_text value "0.2" (at 3.81 2.37 90) (layer "F.Fab")
+    (fp_text value "1" (at 3.81 2.37 90) (layer "F.Fab")
       (effects (font (size 1 1) (thickness 0.15)))
     )
@@
       (effects (font (size 1 1) (thickness 0.15)))
     )
-    (fp_text value "0.2" (at 3.81 2.37) (layer "F.Fab")
+    (fp_text value "1" (at 3.81 2.37) (layer "F.Fab")
       (effects (font (size 1 1) (thickness 0.15)))
     )
@@
       (effects (font (size 1 1) (thickness 0.15)))
     )
-    (fp_text value "0.2" (at 3.81 2.37) (layer "F.Fab")
+    (fp_text value "1" (at 3.81 2.37) (layer "F.Fab")
       (effects (font (size 1 1) (thickness 0.15)))
     )
@@
     (pts (xy 76.2 96.52) (xy 139.7 96.52))
     (height 13.97)
-    (gr_text "63.5000 mm" (at 107.95 108.69) (layer "B.Cu")
+    (gr_text "2500.0000 mils" (at 107.95 108.69) (layer "B.Cu")
       (effects (font (size 1.5 1.5) (thickness 0.3)))
     )
@@
     (pts (xy 203.2 96.52) (xy 203.2 93.98))
     (height 12.7)
-    (gr_text "2.5400 mm" (at 214.75 95.25 90) (layer "Dwgs.User")
+    (gr_text "100.0000 mils" (at 214.75 95.25 90) (layer "Dwgs.User")
       (effects (font (size 1 1) (thickness 0.15)))
     )
@@
     (pts (xy 85.09 96.52) (xy 76.2 96.52))
     (height -8.89)
-    (gr_text "8.8900 mm" (at 80.645 106.68) (layer "Dwgs.User")
+    (gr_text "350.0000 mils" (at 80.645 106.68) (layer "Dwgs.User")
       (effects (font (size 1 1) (thickness 0.15)))
     )
@@
     (pts (xy 76.2 93.98) (xy 76.2 96.52))
     (height 12.7)
-    (gr_text "2.5400 mm" (at 62.35 95.25 90) (layer "Dwgs.User")
+    (gr_text "100.0000 mils" (at 62.35 95.25 90) (layer "Dwgs.User")
       (effects (font (size 1 1) (thickness 0.15)))
     )
@@
     (pts (xy 203.2 96.52) (xy 194.31 96.52))
     (height -8.89)
-    (gr_text "8.8900 mm" (at 198.755 106.68) (layer "Dwgs.User")
-      (effects (font (size 1 1) (thickness 0.15)))
-    )
+    (gr_text "350.0000 mils" (at 198.755 106.68) (layer "Dwgs.User")
+      (effects (font (size 1 1) (thickness 0.15)))
+    )
