File: nixie_main_board/nixie_main_board.kicad_sch (KiCad schematic)
At the start: 48 parts, among them J1 Conn_02x05_Odd_Even, J2 Conn_02x05_Odd_Even, J3 USB_C_Receptacle_USB2.0, J4 Conn_01x02_Male, J5 AVR-ISP-6, J6 Conn_01x01_Male, Q1 BC557, Q2 IRL640, SW1 RotaryEncoder_Switch, SW2 SW_Push, SW3 SW_Push, U1 ATmega328P-PU, U2 MC34063AP, U5 DS3231M, Y1 16 MHz

Commit message: Add title/date/revision
Other:
- title: (none) -> Nixie Clock Main Board
Changed lines of the file:
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@@
 (kicad_sch (version 20211123) (generator eeschema)
   (paper "A4")
+  (title_block
+    (title "Nixie Clock Main Board")
+    (date "2022-01-29")
+    (rev "1")
+  )
   (junction (at 200.66 123.19) (diameter 0) (color 0 0 0 0)
   )

Commit message: Fix sense resistor values
Parts:
- R1, R11, R12, R13, R14: value 0.2 -> 1
Changed lines of the file:
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@@
     (in_bom yes) (on_board yes)
     (property "Reference" "R12" (id 0) (at 63.5 25.4 90))
-    (property "Value" "0.2" (id 1) (at 69.85 26.67 90))
+    (property "Value" "1" (id 1) (at 69.85 26.67 90))
     (property "Footprint" "Resistor_THT:R_Axial_DIN0207_L6.3mm_D2.5mm_P7.62mm_Horizontal" (id 2) (at 69.85 28.448 90)
       (effects (font (size 1.27 1.27)) hide)
@@
     (in_bom yes) (on_board yes)
     (property "Reference" "R14" (id 0) (at 63.5 30.48 90))
-    (property "Value" "0.2" (id 1) (at 69.85 31.75 90))
+    (property "Value" "1" (id 1) (at 69.85 31.75 90))
     (property "Footprint" "Resistor_THT:R_Axial_DIN0207_L6.3mm_D2.5mm_P7.62mm_Horizontal" (id 2) (at 69.85 33.528 90)
       (effects (font (size 1.27 1.27)) hide)
@@
     (in_bom yes) (on_board yes)
     (property "Reference" "R13" (id 0) (at 63.5 27.94 90))
-    (property "Value" "0.2" (id 1) (at 69.85 29.21 90))
+    (property "Value" "1" (id 1) (at 69.85 29.21 90))
     (property "Footprint" "Resistor_THT:R_Axial_DIN0207_L6.3mm_D2.5mm_P7.62mm_Horizontal" (id 2) (at 69.85 30.988 90)
       (effects (font (size 1.27 1.27)) hide)
@@
     (in_bom yes) (on_board yes)
     (property "Reference" "R1" (id 0) (at 63.5 20.32 90))
-    (property "Value" "0.2" (id 1) (at 69.85 21.59 90))
+    (property "Value" "1" (id 1) (at 69.85 21.59 90))
     (property "Footprint" "Resistor_THT:R_Axial_DIN0207_L6.3mm_D2.5mm_P7.62mm_Horizontal" (id 2) (at 69.85 23.368 90)
       (effects (font (size 1.27 1.27)) hide)
@@
     (in_bom yes) (on_board yes)
     (property "Reference" "R11" (id 0) (at 63.5 22.86 90))
-    (property "Value" "0.2" (id 1) (at 69.85 24.13 90))
+    (property "Value" "1" (id 1) (at 69.85 24.13 90))
     (property "Footprint" "Resistor_THT:R_Axial_DIN0207_L6.3mm_D2.5mm_P7.62mm_Horizontal" (id 2) (at 69.85 25.908 90)
       (effects (font (size 1.27 1.27)) hide)
@@
     )
     (path "/415ccd57-f96d-472d-9848-b21d1712e51d"
-      (reference "R1") (unit 1) (value "0.2") (footprint "Resistor_THT:R_Axial_DIN0207_L6.3mm_D2.5mm_P7.62mm_Horizontal")
+      (reference "R1") (unit 1) (value "1") (footprint "Resistor_THT:R_Axial_DIN0207_L6.3mm_D2.5mm_P7.62mm_Horizontal")
     )
     (path "/5936c555-55c8-4d29-9c16-3c94f395520e"
@@
     )
     (path "/76bb146a-eb83-404e-a172-7459e040eeed"
-      (reference "R11") (unit 1) (value "0.2") (footprint "Resistor_THT:R_Axial_DIN0207_L6.3mm_D2.5mm_P7.62mm_Horizontal")
+      (reference "R11") (unit 1) (value "1") (footprint "Resistor_THT:R_Axial_DIN0207_L6.3mm_D2.5mm_P7.62mm_Horizontal")
     )
     (path "/35683364-681c-4c21-870f-ce79f3a9eb54"
-      (reference "R12") (unit 1) (value "0.2") (footprint "Resistor_THT:R_Axial_DIN0207_L6.3mm_D2.5mm_P7.62mm_Horizontal")
+      (reference "R12") (unit 1) (value "1") (footprint "Resistor_THT:R_Axial_DIN0207_L6.3mm_D2.5mm_P7.62mm_Horizontal")
     )
     (path "/3e70ae01-7d52-43d8-ae16-440033540130"
-      (reference "R13") (unit 1) (value "0.2") (footprint "Resistor_THT:R_Axial_DIN0207_L6.3mm_D2.5mm_P7.62mm_Horizontal")
+      (reference "R13") (unit 1) (value "1") (footprint "Resistor_THT:R_Axial_DIN0207_L6.3mm_D2.5mm_P7.62mm_Horizontal")
     )
     (path "/3582bb59-3d94-4693-b9cc-99590cd0046f"
-      (reference "R14") (unit 1) (value "0.2") (footprint "Resistor_THT:R_Axial_DIN0207_L6.3mm_D2.5mm_P7.62mm_Horizontal")
+      (reference "R14") (unit 1) (value "1") (footprint "Resistor_THT:R_Axial_DIN0207_L6.3mm_D2.5mm_P7.62mm_Horizontal")
     )
     (path "/18b0f152-f58f-4834-9ff3-bf4365b64b41"
